File: hw/sch_pcb/RFSWITCH01A.kicad_pcb (KiCad board)
At the start: 2 copper layers, 40.1 x 40.1 mm, 45 parts, among them J1 HEADER_2x03_PARALLEL, J10 HEADER_2x01_PARALLEL, J2 SMA, J3 SMA, J4 HEADER_2x01_PARALLEL, J5 HEADER_2x01_PARALLEL, J6 HEADER_2x01_PARALLEL, J7 SMA, J8 SMA, J9 HEADER_2x01_PARALLEL, M1 HOLE, M2 HOLE, M3 HOLE, M4 HOLE, U1 TPS22945DCKR, U2 PE4259, U3 SPF5189Z, U4 PE4259

Commit message: Cleanup silkscreen.
Routing:
- net GND: vias 276 -> 283
Changed lines of the file:
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@@
     (property "Sheet file" "C:/Chroust/stare/MLAB_G/Moduly_zvlast/RFSWITCH01/hw/sch_pcb/RFSWITCH01A.kicad_sch")
     (attr smd)
-    (fp_text reference "U4" (at 0 2) (layer "B.SilkS")
+    (fp_text reference "U4" (at 1.4224 -2.032) (layer "B.SilkS")
       (effects (font (size 1 1) (thickness 0.15)) (justify mirror))
     )
@@
     (property "Sheet file" "C:/Chroust/stare/MLAB_G/Moduly_zvlast/RFSWITCH01/hw/sch_pcb/RFSWITCH01A.kicad_sch")
     (attr smd)
-    (fp_text reference "U3" (at 0.3 3.5) (layer "B.SilkS")
+    (fp_text reference "U3" (at -3.8354 -0.4064 90) (layer "B.SilkS")
       (effects (font (size 1 1) (thickness 0.15)) (justify mirror))
     )
@@
     (property "UST_ID" "5c70984512875079b91f88b1")
     (attr smd)
-    (fp_text reference "D3" (at 0 2 -270) (layer "B.SilkS")
+    (fp_text reference "D3" (at -1.6536 1.8796 -270) (layer "B.SilkS")
       (effects (font (size 1 1) (thickness 0.15)) (justify mirror))
     )
@@
     (property "Sheet file" "C:/Chroust/stare/MLAB_G/Moduly_zvlast/RFSWITCH01/hw/sch_pcb/RFSWITCH01A.kicad_sch")
     (attr smd)
-    (fp_text reference "U1" (at 0 2) (layer "B.SilkS")
+    (fp_text reference "U1" (at 2.4638 -2.0828) (layer "B.SilkS")
       (effects (font (size 1 1) (thickness 0.15)) (justify mirror))
     )
@@
     (property "Sheet file" "C:/Chroust/stare/MLAB_G/Moduly_zvlast/RFSWITCH01/hw/sch_pcb/RFSWITCH01A.kicad_sch")
     (attr smd)
-    (fp_text reference "L1" (at 0 1.55) (layer "B.SilkS")
+    (fp_text reference "L1" (at 2.3579 0.889) (layer "B.SilkS")
       (effects (font (size 1 1) (thickness 0.15)) (justify mirror))
     )
@@
     (property "Sheet file" "C:/Chroust/stare/MLAB_G/Moduly_zvlast/RFSWITCH01/hw/sch_pcb/RFSWITCH01A.kicad_sch")
     (attr through_hole)
-    (fp_text reference "FL1" (at -1.016 3.556) (layer "B.SilkS")
+    (fp_text reference "FL1" (at 1.3716 -2.794) (layer "B.SilkS")
       (effects (font (size 1 1) (thickness 0.15)) (justify mirror))
     )
@@
     (property "Sheet file" "C:/Chroust/stare/MLAB_G/Moduly_zvlast/RFSWITCH01/hw/sch_pcb/RFSWITCH01A.kicad_sch")
     (attr smd)
-    (fp_text reference "U2" (at 0 2) (layer "B.SilkS")
+    (fp_text reference "U2" (at 1.8542 2.032) (layer "B.SilkS")
       (effects (font (size 1 1) (thickness 0.15)) (justify mirror))
     )
@@
     (property "UST_ID" "5c70984512875079b91f88b1")
     (attr smd)
-    (fp_text reference "D2" (at 0 2 -270) (layer "B.SilkS")
+    (fp_text reference "D2" (at -1.586685 -1.822101 -270) (layer "B.SilkS")
       (effects (font (size 1 1) (thickness 0.15)) (justify mirror))
     )
@@
     (property "Sheet file" "C:/Chroust/stare/MLAB_G/Moduly_zvlast/RFSWITCH01/hw/sch_pcb/RFSWITCH01A.kicad_sch")
     (attr smd)
-    (fp_text reference "L3" (at 0 1.55) (layer "B.SilkS")
+    (fp_text reference "L3" (at -1.8753 1.6764) (layer "B.SilkS")
       (effects (font (size 1 1) (thickness 0.15)) (justify mirror))
     )
@@
   (via (at 20.1676 -10.0965) (size 0.45) (drill 0.2) (layers "F.Cu" "B.Cu") (net 2))
   (via (at 15.1384 -14.3256) (size 0.45) (drill 0.2) (layers "F.Cu" "B.Cu") (net 2))
+  (via (at 8.89 -20.2692) (size 0.45) (drill 0.2) (layers "F.Cu" "B.Cu") (net 2))
   (via (at 23.4188 -21.2344) (size 0.45) (drill 0.2) (layers "F.Cu" "B.Cu") (net 2))
   (via (at 13.8176 -21.0312) (size 0.45) (drill 0.2) (layers "F.Cu" "B.Cu") (net 2))
@@
   (via (at 21.0312 -15.0876) (size 0.45) (drill 0.2) (layers "F.Cu" "B.Cu") (net 2))
   (via (at 22.8092 -29.3624) (size 0.45) (drill 0.2) (layers "F.Cu" "B.Cu") (net 2))
-  (via (at 22.606 -11.0236) (size 0.45) (drill 0.2) (layers "F.Cu" "B.Cu") (net 2))
+  (via (at 22.86 -11.0236) (size 0.45) (drill 0.2) (layers "F.Cu" "B.Cu") (net 2))
   (via (at 12.4968 -15.113) (size 0.45) (drill 0.2) (layers "F.Cu" "B.Cu") (net 2))
   (via (at 14.8844 -9.7536) (size 0.45) (drill 0.2) (layers "F.Cu" "B.Cu") (net 2))
@@
   (via (at 16.6624 -14.8844) (size 0.45) (drill 0.2) (layers "F.Cu" "B.Cu") (net 2))
   (via (at 35.8648 -14.478) (size 0.45) (drill 0.2) (layers "F.Cu" "B.Cu") (net 2))
-  (via (at 21.9964 -11.0236) (size 0.45) (drill 0.2) (layers "F.Cu" "B.Cu") (net 2))
+  (via (at 22.1488 -11.0236) (size 0.45) (drill 0.2) (layers "F.Cu" "B.Cu") (net 2))
   (via (at 18.6944 -21.4884) (size 0.45) (drill 0.2) (layers "F.Cu" "B.Cu") (net 2))
   (via (at 28.956 -11.5316) (size 0.45) (drill 0.2) (layers "F.Cu" "B.Cu") (net 2))
@@
   (via (at 24.0792 -17.8308) (size 0.45) (drill 0.2) (layers "F.Cu" "B.Cu") (net 2))
   (via (at 29.8704 -13.716) (size 0.45) (drill 0.2) (layers "F.Cu" "B.Cu") (net 2))
+  (via (at 37.5412 -20.574) (size 0.45) (drill 0.2) (layers "F.Cu" "B.Cu") (net 2))
   (via (at 25.9588 -20.3708) (size 0.45) (drill 0.2) (layers "F.Cu" "B.Cu") (net 2))
   (via (at 26.7208 -14.8336) (size 0.45) (drill 0.2) (layers "F.Cu" "B.Cu") (net 2))
@@
   (via (at 28.0924 -16.1544) (size 0.45) (drill 0.2) (layers "F.Cu" "B.Cu") (net 2))
   (via (at 34.6964 -24.5364) (size 0.45) (drill 0.2) (layers "F.Cu" "B.Cu") (net 2))
+  (via (at 2.9464 -20.6756) (size 0.45) (drill 0.2) (layers "F.Cu" "B.Cu") (net 2))
   (via (at 10.3124 -24.7396) (size 0.45) (drill 0.2) (layers "F.Cu" "B.Cu") (net 2))
   (via (at 7.1628 -15.9512) (size 0.45) (drill 0.2) (layers "F.Cu" "B.Cu") (net 2))
@@
   (via (at 9.906 -26.8224) (size 0.45) (drill 0.2) (layers "F.Cu" "B.Cu") (net 2))
   (via (at 20.1676 -10.7188) (size 0.45) (drill 0.2) (layers "F.Cu" "B.Cu") (net 2))
+  (via (at 33.1216 -19.812) (size 0.45) (drill 0.2) (layers "F.Cu" "B.Cu") (net 2))
   (via (at 4.7752 -14.732) (size 0.45) (drill 0.2) (layers "F.Cu" "B.Cu") (net 2))
   (via (at 18.2372 -12.8016) (size 0.45) (drill 0.2) (layers "F.Cu" "B.Cu") (net 2))
@@
   (via (at 28.0924 -21.336) (size 0.45) (drill 0.2) (layers "F.Cu" "B.Cu") (net 2))
   (via (at 35.6616 -13.8684) (size 0.45) (drill 0.2) (layers "F.Cu" "B.Cu") (net 2))
+  (via (at 26.3144 -11.8364) (size 0.45) (drill 0.2) (layers "F.Cu" "B.Cu") (net 2))
   (via (at 33.8836 -16.1544) (size 0.45) (drill 0.2) (layers "F.Cu" "B.Cu") (net 2))
   (via (at 18.6436 -14.0208) (size 0.45) (drill 0.2) (layers "F.Cu" "B.Cu") (net 2))
+  (via (at 29.21 -9.3472) (size 0.45) (drill 0.2) (layers "F.Cu" "B.Cu") (net 2))
   (via (at 19.7104 -18.1864) (size 0.45) (drill 0.2) (layers "F.Cu" "B.Cu") (net 2))
   (via (at 29.0068 -13.716) (size 0.45) (drill 0.2) (layers "F.Cu" "B.Cu") (net 2))
@@
   (via (at 13.716 -14.605) (size 0.45) (drill 0.2) (layers "F.Cu" "B.Cu") (net 2))
   (via (at 13.5128 -23.9268) (size 0.45) (drill 0.2) (layers "F.Cu" "B.Cu") (net 2))
+  (via (at 21.4884 -22.86) (size 0.45) (drill 0.2) (layers "F.Cu" "B.Cu") (net 2))
   (via (at 17.1704 -17.1704) (size 0.45) (drill 0.2) (layers "F.Cu" "B.Cu") (net 2))
   (via (at 18.6944 -19.1008) (size 0.45) (drill 0.2) (layers "F.Cu" "B.Cu") (net 2))
@@
   (via (at 34.4932 -27.5844) (size 0.45) (drill 0.2) (layers "F.Cu" "B.Cu") (net 2))
   (via (at 26.3652 -25.6032) (size 0.45) (drill 0.2) (layers "F.Cu" "B.Cu") (net 2))
-  (via (at 22.86 -11.5824) (size 0.45) (drill 0.2) (layers "F.Cu" "B.Cu") (net 2))
+  (via (at 22.9108 -11.6332) (size 0.45) (drill 0.2) (layers "F.Cu" "B.Cu") (net 2))
   (via (at 28.1432 -24.0792) (size 0.45) (drill 0.2) (layers "F.Cu" "B.Cu") (net 2))
   (via (at 35.8648 -25.908) (size 0.45) (drill 0.2) (layers "F.Cu" "B.Cu") (net 2))
@@
   (segment (start 16.89 -11.43) (end 17.492786 -11.43) (width 0.861) (layer "B.Cu") (net 5))
   (arc (start 18.199893 -11.137107) (mid 17.87547 -11.35388) (end 17.492786 -11.43) (width 0.861) (layer "B.Cu") (net 5))
-  (segment (start 23.875 -12.47) (end 23.875 -10.693694) (width 0.861) (layer "B.Cu") (net 6))
-  (segment (start 21.1455 -10.0965) (end 23.277806 -10.0965) (width 0.861) (layer "B.Cu") (net 6))
-  (segment (start 23.875 -10.693694) (end 23.531099 -10.349793) (width 0.861) (layer "B.Cu") (net 6))
-  (segment (start 23.277806 -10.0965) (end 23.531099 -10.349793) (width 0.861) (layer "B.Cu") (net 6))
+  (segment (start 23.875 -12.47) (end 23.875 -11.107908) (width 0.861) (layer "B.Cu") (net 6))
+  (segment (start 21.1455 -10.0965) (end 22.946435 -10.0965) (width 0.861) (layer "B.Cu") (net 6))
+  (segment (start 23.582107 -10.400801) (end 23.531099 -10.349793) (width 0.861) (layer "B.Cu") (net 6))
+  (segment (start 23.51212 -10.330814) (end 23.531099 -10.349793) (width 0.861) (layer "B.Cu") (net 6))
+  (arc (start 23.875 -11.107908) (mid 23.79888 -10.725225) (end 23.582107 -10.400801) (width 0.861) (layer "B.Cu") (net 6))
+  (arc (start 22.946435 -10.0965) (mid 23.252581 -10.157396) (end 23.51212 -10.330814) (width 0.861) (layer "B.Cu") (net 6))
   (segment (start 26.924 -22.783179) (end 26.924 -21.336) (width 0.861) (layer "B.Cu") (net 7))
   (segment (start 26.929992 -22.789171) (end 26.924 -22.783179) (width 0.861) (layer "B.Cu") (net 7))
